File: display-module/LED-display_x4.kicad_pcb (KiCad board)
At the start: 2 copper layers, 61 x 29.2 mm, 8 parts, among them J1 Conn_DP1, J2 Conn_DP1, M1 Conn_01x01, M2 Conn_01x01, M3 Conn_01x01, M4 Conn_01x01

Commit message: update file
I make mistake in schematics library & footprint library
now devices are correct, I divided 7 segment display at
two separate CA & CC

bye!
Parts:
- D1, D2: value HDSP-5623 -> HDSP-5623-CA
