File: voltmeter/file5ECBC5A0.sch (KiCad schematic (older format))
At the start: 5 parts, among them U4 4069

Commit message: update file
I make mistake in schematics library & footprint library
now devices are correct, I divided 7 segment display at
two separate CA & CC

bye!
Parts:
- renumbered D2 to D7
Changed lines of the file:
@@
 $EndDescr
 $Comp
-L Diode:1N914 D2
+L Diode:1N914 D7
 U 1 1 5ECB70C6
 P 6500 2800
-F 0 "D2" V 6454 2880 50  0000 L CNN
+F 0 "D7" V 6454 2880 50  0000 L CNN
 F 1 "1N914" V 6545 2880 50  0000 L CNN
 F 2 "Diode_THT:D_DO-35_SOD27_P7.62mm_Horizontal" H 6500 2625 50  0001 C CNN
@@
 V-
 $Comp
-L power:GND #PWR0101
+L power:GND #PWR04
 U 1 1 5ECD026B
 P 6750 2350
-F 0 "#PWR0101" H 6750 2100 50  0001 C CNN
+F 0 "#PWR04" H 6750 2100 50  0001 C CNN
 F 1 "GND" H 6755 2177 50  0000 C CNN
 F 2 "" H 6750 2350 50  0001 C CNN
@@
 $EndComp
 $Comp
-L power:GND #PWR0102
+L power:GND #PWR03
 U 1 1 5ECD1B24
 P 3750 3550
-F 0 "#PWR0102" H 3750 3300 50  0001 C CNN
+F 0 "#PWR03" H 3750 3300 50  0001 C CNN
 F 1 "GND" H 3755 3377 50  0000 C CNN
 F 2 "" H 3750 3550 50  0001 C CNN

Commit message: update file
poprawiłem schemat i ponownie wygenerowałem pliki Gerber

I corrected the diagram and re-generated the Gerber files
Parts:
- renumbered D8 to D10, D7 to D9
Changed lines of the file:
@@
 $EndDescr
 $Comp
-L Diode:1N914 D7
+L Diode:1N914 D9
 U 1 1 5ECB70C6
 P 6500 2800
-F 0 "D7" V 6454 2880 50  0000 L CNN
+F 0 "D9" V 6454 2880 50  0000 L CNN
 F 1 "1N914" V 6545 2880 50  0000 L CNN
 F 2 "Diode_THT:D_DO-35_SOD27_P7.62mm_Horizontal" H 6500 2625 50  0001 C CNN
@@
 $EndComp
 $Comp
-L Diode:1N914 D8
+L Diode:1N914 D10
 U 1 1 5ECB783B
 P 6500 4150
-F 0 "D8" V 6454 4230 50  0000 L CNN
+F 0 "D10" V 6454 4230 50  0000 L CNN
 F 1 "1N914" V 6545 4230 50  0000 L CNN
 F 2 "Diode_THT:D_DO-35_SOD27_P7.62mm_Horizontal" H 6500 3975 50  0001 C CNN
@@
 V-
 $Comp
-L power:GND #PWR05
+L power:GND #PWR07
 U 1 1 5ECD026B
 P 6750 2350
-F 0 "#PWR05" H 6750 2100 50  0001 C CNN
+F 0 "#PWR07" H 6750 2100 50  0001 C CNN
 F 1 "GND" H 6755 2177 50  0000 C CNN
 F 2 "" H 6750 2350 50  0001 C CNN
@@
 $EndComp
 $Comp
-L power:GND #PWR04
+L power:GND #PWR06
 U 1 1 5ECD1B24
 P 3750 3550
-F 0 "#PWR04" H 3750 3300 50  0001 C CNN
+F 0 "#PWR06" H 3750 3300 50  0001 C CNN
 F 1 "GND" H 3755 3377 50  0000 C CNN
 F 2 "" H 3750 3550 50  0001 C CNN

Commit message: upload modified file
Connections:
- net labels added: +5V, -5V
- net labels removed: V+
Changed lines of the file:
@@
 Wire Wire Line
 	3900 4500 3500 4500
-Text Label 3600 4500 0    50   ~ 0
-OSC3
 Wire Wire Line
 	6750 4500 6750 4900
@@
 Wire Wire Line
 	3750 2400 3750 2200
-Text Label 3750 2300 0    50   ~ 0
-V+
 Wire Wire Line
 	3750 3400 3750 3550
@@
 Wire Wire Line
 	6500 3500 6500 4000
+$Comp
+L power:+5V #PWR?
+U 1 1 5F2EEE2B
+P 3750 2200
+F 0 "#PWR?" H 3750 2050 50  0001 C CNN
+F 1 "+5V" H 3765 2373 50  0000 C CNN
+F 2 "" H 3750 2200 50  0001 C CNN
+F 3 "" H 3750 2200 50  0001 C CNN
+	1    3750 2200
+	1    0    0    -1
+$EndComp
+$Comp
+L power:-5V #PWR?
+U 1 1 5F2EF5C3
+P 6750 4900
+F 0 "#PWR?" H 6750 5000 50  0001 C CNN
+F 1 "-5V" H 6765 5073 50  0000 C CNN
+F 2 "" H 6750 4900 50  0001 C CNN
+F 3 "" H 6750 4900 50  0001 C CNN
+	1    6750 4900
+	-1   0    0    1
+$EndComp
+Text GLabel 3500 4500 0    50   Input ~ 0
+OSC3
 $EndSCHEMATC
